File: charger/charger.sch (KiCad schematic (older format))
At the start: 92 parts, among them U1 MSP432, U2 NCP718xSN500

Commit message: add footprints
Parts:
- added C21, C29: 0.1 uF, Capacitor_SMD:C_1206_3216Metric, symbol Device:C
- added J2, J3: Conn_01x06, Connector_PinHeader_2.54mm:PinHeader_1x06_P2.54mm_Vertical, symbol Connector_Generic:Conn_01x06
- added J4: Conn_01x03, Connector_PinHeader_2.54mm:PinHeader_1x03_P2.54mm_Vertical, symbol Connector_Generic:Conn_01x03
- added R1, R10, R7, R8, R9: 205, Resistor_SMD:R_1206_3216Metric, symbol Device:R_US
- added R11, R2, R23: 1k, Resistor_SMD:R_1206_3216Metric, symbol Device:R_US
- C1, C2: footprint (none) -> Capacitor_SMD:C_1206_3216Metric
- C10, C11, C12, C13, C14, C15, C16, C17, C18, C19, C20, C22, C23, C24, C26, C27, C28, C3, C30, C32, C33, C34, C35, C6, C7, C8, C9: renamed from C?; footprint (none) -> Capacitor_SMD:C_1206_3216Metric
- C25: renamed from C?; footprint (none) -> Capacitor_THT:CP_Radial_D30.0mm_P10.00mm_SnapIn
- C31: renamed from C?; footprint (none) -> Capacitor_THT:CP_Radial_D5.0mm_P2.00mm
- C36: renamed from C?; footprint (none) -> Capacitor_THT:CP_Radial_D6.3mm_P2.50mm
- C4, C5: renamed from C?; footprint (none) -> Capacitor_THT:CP_Radial_D25.0mm_P10.00mm_SnapIn
- D1, D2, D3, D4, D5: renamed from D?; footprint (none) -> Diode_SMD:D_SMA
- FB1, FB2: renamed from FB?; footprint (none) -> Inductor_SMD:L_0805_2012Metric
- J1: renamed from J?; footprint (none) -> Connector_PinHeader_2.54mm:PinHeader_1x06_P2.54mm_Vertical
- J5: renamed from J?; footprint (none) -> Connector_PinHeader_2.54mm:PinHeader_1x02_P2.54mm_Vertical
- L1, L2: renamed from L?; footprint (none) -> MWD_Footprints:7443642200 _Inductor
- U3: renamed from U?; footprint (none) -> Package_TO_SOT_SMD:SOT-23-5
- gave numbers to parts that had none: 44
Connections:
- net +5V: no longer U1.11 (5V)
- net GND: now also C21.2, C29.2, J2.6 (Pin_6), J3.6 (Pin_6), J4.3 (Pin_3); no longer U1.12 (GND)
- net I_bat: now also R23.1
- net I_in: now also R11.1
- net Input_EN: now also U1.40 (P3.6), R1.1; no longer U3.3
- net PWM_H1: now also R9.1
- net PWM_H2: now also R10.1
- net PWM_L1: now also R7.1
- net PWM_L2: now also R8.1
- net V_bat_sense: now also U1.16 (P4.4), J2.3 (Pin_3)
- net V_in_sense: now also U1.15 (P4.2), J2.1 (Pin_1)
- net I2C_SDA: now reaches U1.10 (P6.4)
- net I2C_SDA: now also J4.2 (Pin_2)
- net I_in_sense: now reaches U1.13 (P6.1)
- net I_in_sense: now also C21.1, J2.2 (Pin_2), R11.2
- net I_bat_sense: now reaches U1.14 (P4.0)
- net I_bat_sense: now also C29.1, J2.4 (Pin_4), R23.2
- net G2_L: now reaches U1.21 (P2.7)
- net G2_L: now also R8.2
- net G2_H: now reaches U1.22 (P2.6)
- net G2_H: now also R10.2
- net G1_H: now reaches U1.23 (P2.4)
- net G1_H: now also R9.2
- net G1_L: now reaches U1.32 (P2.5)
- net G1_L: now also R7.2
- net SPI_CS_WL: now reaches U1.33 (P3.0)
- net SPI_CS_WL: now also J3.2 (Pin_2)
- net SPI_MOSI: now reaches U1.36 (P1.6)
- net SPI_MOSI: now also J3.3 (Pin_3)
- net SPI_MISO: now reaches U1.37 (P1.7)
- net SPI_MISO: now also J3.4 (Pin_4)
- net SPI_CS_D: now reaches U1.38 (P5.0)
- net SPI_CS_D: now also J3.5 (Pin_5)
- net SPI_CLK: now reaches U1.7 (P1.5)
- net SPI_CLK: now also J3.1 (Pin_1)
- net at U1.8 (P4.6): now also R2.2
- net I2C_SCL: now reaches U1.9 (P6.5)
- net I2C_SCL: now also J4.1 (Pin_1)
- new net: R1.2, U3.3
- new net misc_signal: J2.5 (Pin_5), R2.1

Commit message: start on pcb
Parts:
- D6: footprint (none) -> Diode_SMD:D_SMB
- L3: footprint (none) -> Inductor_SMD:L_Bourns_SRR1260
- TP1, TP2, TP3, TP4, TP5, TP6, TP7: footprint (none) -> Connector_Pin:Pin_D1.4mm_L8.5mm_W2.8mm_FlatFork
Connections:
- net V_p is gone; now on net V_in: C30.2, R25.2, U8.8 (VIN)
Other:
- moved on the sheet: C1, C2, R27, TP5, TP7, U2
Changed lines of the file:
@@
 L Regulator_Linear:NCP718xSN500 U2
 U 1 1 5EBB340C
-P 10150 1150
-F 0 "U2" H 10150 1517 50  0000 C CNN
-F 1 "NCP718xSN500" H 10150 1426 50  0000 C CNN
-F 2 "Package_TO_SOT_SMD:SOT-23-5" H 10150 1500 50  0001 C CNN
-F 3 "https://www.onsemi.com/pub/Collateral/NCP718-D.PDF" H 10150 1650 50  0001 C CNN
-	1    10150 1150
+P 10000 1150
+F 0 "U2" H 10000 1517 50  0000 C CNN
+F 1 "NCP718xSN500" H 10000 1426 50  0000 C CNN
+F 2 "Package_TO_SOT_SMD:SOT-23-5" H 10000 1500 50  0001 C CNN
+F 3 "https://www.onsemi.com/pub/Collateral/NCP718-D.PDF" H 10000 1650 50  0001 C CNN
+	1    10000 1150
 	1    0    0    -1
 $EndComp
@@
 L power:+5V #PWR02
 U 1 1 5EBB5145
-P 10750 950
-F 0 "#PWR02" H 10750 800 50  0001 C CNN
-F 1 "+5V" H 10765 1123 50  0000 C CNN
-F 2 "" H 10750 950 50  0001 C CNN
-F 3 "" H 10750 950 50  0001 C CNN
-	1    10750 950
+P 10600 950
+F 0 "#PWR02" H 10600 800 50  0001 C CNN
+F 1 "+5V" H 10615 1123 50  0000 C CNN
+F 2 "" H 10600 950 50  0001 C CNN
+F 3 "" H 10600 950 50  0001 C CNN
+	1    10600 950
 	1    0    0    -1
 $EndComp
@@
 L Device:C_Small C1
 U 1 1 5EBBA522
-P 9500 1550
-F 0 "C1" H 9592 1596 50  0000 L CNN
-F 1 "1 uF" H 9592 1505 50  0000 L CNN
-F 2 "Capacitor_SMD:C_1206_3216Metric" H 9500 1550 50  0001 C CNN
-F 3 "~" H 9500 1550 50  0001 C CNN
-	1    9500 1550
+P 9350 1550
+F 0 "C1" H 9442 1596 50  0000 L CNN
+F 1 "1 uF" H 9442 1505 50  0000 L CNN
+F 2 "Capacitor_SMD:C_1206_3216Metric" H 9350 1550 50  0001 C CNN
+F 3 "~" H 9350 1550 50  0001 C CNN
+	1    9350 1550
 	1    0    0    -1
 $EndComp
@@
 L Device:C_Small C2
 U 1 1 5EBBB602
-P 10750 1200
-F 0 "C2" H 10842 1246 50  0000 L CNN
-F 1 "1 uF" H 10842 1155 50  0000 L CNN
-F 2 "Capacitor_SMD:C_1206_3216Metric" H 10750 1200 50  0001 C CNN
-F 3 "~" H 10750 1200 50  0001 C CNN
-	1    10750 1200
+P 10600 1200
+F 0 "C2" H 10692 1246 50  0000 L CNN
+F 1 "1 uF" H 10692 1155 50  0000 L CNN
+F 2 "Capacitor_SMD:C_1206_3216Metric" H 10600 1200 50  0001 C CNN
+F 3 "~" H 10600 1200 50  0001 C CNN
+	1    10600 1200
 	1    0    0    -1
 $EndComp
@@
 L power:GND #PWR050
 U 1 1 5EBBBBA3
-P 10150 1600
-F 0 "#PWR050" H 10150 1350 50  0001 C CNN
-F 1 "GND" H 10155 1427 50  0000 C CNN
-F 2 "" H 10150 1600 50  0001 C CNN
-F 3 "" H 10150 1600 50  0001 C CNN
-	1    10150 1600
-	1    0    0    -1
-$EndComp
-Wire Wire Line
-	10150 1600 10150 1450
-Connection ~ 10150 1450
-Wire Wire Line
-	10750 1300 10750 1450
-Wire Wire Line
-	10750 1450 10150 1450
-Wire Wire Line
-	10450 1050 10750 1050
-Wire Wire Line
-	10750 1050 10750 950
-Wire Wire Line
-	10750 1100 10750 1050
-Connection ~ 10750 1050
+P 10000 1600
+F 0 "#PWR050" H 10000 1350 50  0001 C CNN
+F 1 "GND" H 10005 1427 50  0000 C CNN
+F 2 "" H 10000 1600 50  0001 C CNN
+F 3 "" H 10000 1600 50  0001 C CNN
+	1    10000 1600
+	1    0    0    -1
+$EndComp
+Wire Wire Line
+	10000 1600 10000 1450
+Connection ~ 10000 1450
+Wire Wire Line
+	10600 1300 10600 1450
+Wire Wire Line
+	10600 1450 10000 1450
+Wire Wire Line
+	10300 1050 10600 1050
+Wire Wire Line
+	10600 1050 10600 950
+Wire Wire Line
+	10600 1100 10600 1050
+Connection ~ 10600 1050
 $Comp
 L Device:R_Small_US R27
 U 1 1 5EBBCB90
-P 9650 1150
-F 0 "R27" V 9855 1150 50  0000 C CNN
-F 1 "0 ohm" V 9764 1150 50  0000 C CNN
-F 2 "Resistor_SMD:R_1206_3216Metric" H 9650 1150 50  0001 C CNN
-F 3 "~" H 9650 1150 50  0001 C CNN
-	1    9650 1150
-	0    1    1    0
-$EndComp
-Wire Wire Line
-	9500 900  9500 1050
-Wire Wire Line
-	9500 1050 9850 1050
-Wire Wire Line
-	9850 1150 9750 1150
-Wire Wire Line
-	9500 1450 9500 1150
-Connection ~ 9500 1050
-Wire Wire Line
-	9550 1150 9500 1150
-Connection ~ 9500 1150
-Wire Wire Line
-	9500 1150 9500 1050
+P 9500 1150
+F 0 "R27" V 9705 1150 50  0000 C CNN
+F 1 "0 ohm" V 9614 1150 50  0000 C CNN
+F 2 "Resistor_SMD:R_1206_3216Metric" H 9500 1150 50  0001 C CNN
+F 3 "~" H 9500 1150 50  0001 C CNN
+	1    9500 1150
+	0    1    1    0
+$EndComp
+Wire Wire Line
+	9350 900  9350 1050
+Wire Wire Line
+	9350 1050 9700 1050
+Wire Wire Line
+	9700 1150 9600 1150
+Wire Wire Line
+	9350 1450 9350 1150
+Connection ~ 9350 1050
+Wire Wire Line
+	9400 1150 9350 1150
+Connection ~ 9350 1150
+Wire Wire Line
+	9350 1150 9350 1050
 $Comp
 L power:GND #PWR049
 U 1 1 5EBC9AAB
-P 9500 1700
-F 0 "#PWR049" H 9500 1450 50  0001 C CNN
-F 1 "GND" H 9505 1527 50  0000 C CNN
-F 2 "" H 9500 1700 50  0001 C CNN
-F 3 "" H 9500 1700 50  0001 C CNN
-	1    9500 1700
-	1    0    0    -1
-$EndComp
-Wire Wire Line
-	9500 1650 9500 1700
+P 9350 1700
+F 0 "#PWR049" H 9350 1450 50  0001 C CNN
+F 1 "GND" H 9355 1527 50  0000 C CNN
+F 2 "" H 9350 1700 50  0001 C CNN
+F 3 "" H 9350 1700 50  0001 C CNN
+	1    9350 1700
+	1    0    0    -1
+$EndComp
+Wire Wire Line
+	9350 1650 9350 1700
 $Comp
 L power:+5V #PWR046
@@
 L power:+10V #PWR048
 U 1 1 5ED3013A
-P 9500 900
-F 0 "#PWR048" H 9500 750 50  0001 C CNN
-F 1 "+10V" H 9515 1073 50  0000 C CNN
-F 2 "" H 9500 900 50  0001 C CNN
-F 3 "" H 9500 900 50  0001 C CNN
-	1    9500 900
+P 9350 900
+F 0 "#PWR048" H 9350 750 50  0001 C CNN
+F 1 "+10V" H 9365 1073 50  0000 C CNN
+F 2 "" H 9350 900 50  0001 C CNN
+F 3 "" H 9350 900 50  0001 C CNN
+	1    9350 900
 	1    0    0    -1
 $EndComp
@@
 Wire Wire Line
 	8650 4050 8750 4050
-Text Label 8650 3950 0    50   ~ 0
-V_p
 $Comp
 L Device:C C30
@@
 F 0 "L3" V 10590 4250 50  0000 C CNN
 F 1 "220 uH" V 10499 4250 50  0000 C CNN
-F 2 "" H 10400 4250 50  0001 C CNN
-F 3 "~" H 10400 4250 50  0001 C CNN
+F 2 "Inductor_SMD:L_Bourns_SRR1260" H 10400 4250 50  0001 C CNN
+F 3 "https://www.mouser.com/ProductDetail/Bourns/SRR1260-221K?qs=sGAEpiMZZMv126LJFLh8y2g1MQW3KQGurY%2FzTCT0qxM%3D" H 10400 4250 50  0001 C CNN
 	1    10400 4250
 	0    -1   -1   0
@@
 F 0 "D6" V 10004 4729 50  0000 L CNN
 F 1 "B1100B" V 10095 4729 50  0000 L CNN
-F 2 "" H 10050 4650 50  0001 C CNN
-F 3 "~" H 10050 4650 50  0001 C CNN
+F 2 "Diode_SMD:D_SMB" H 10050 4650 50  0001 C CNN
+F 3 "https://www.digikey.com/en/products/detail/diodes-incorporated/B1100B-13-F/768766" H 10050 4650 50  0001 C CNN
 	1    10050 4650
 	0    1    1    0
@@
 L Connector:TestPoint TP5
 U 1 1 5F1C5256
-P 9500 1050
-F 0 "TP5" V 9695 1122 50  0000 C CNN
-F 1 "TestPoint" V 9604 1122 50  0000 C CNN
-F 2 "" H 9700 1050 50  0001 C CNN
-F 3 "~" H 9700 1050 50  0001 C CNN
-	1    9500 1050
+P 9350 1050
+F 0 "TP5" V 9545 1122 50  0000 C CNN
+F 1 "TestPoint" V 9454 1122 50  0000 C CNN
+F 2 "Connector_Pin:Pin_D1.4mm_L8.5mm_W2.8mm_FlatFork" H 9550 1050 50  0001 C CNN
+F 3 "~" H 9550 1050 50  0001 C CNN
+	1    9350 1050
 	0    -1   -1   0
 $EndComp
@@
 L Connector:TestPoint TP7
 U 1 1 5F1DAE48
-P 10750 1050
-F 0 "TP7" V 10704 1238 50  0000 L CNN
-F 1 "TestPoint" V 10795 1238 50  0000 L CNN
-F 2 "" H 10950 1050 50  0001 C CNN
-F 3 "~" H 10950 1050 50  0001 C CNN
-	1    10750 1050
+P 10600 1050
+F 0 "TP7" V 10554 1238 50  0000 L CNN
+F 1 "TestPoint" V 10645 1238 50  0000 L CNN
+F 2 "Connector_Pin:Pin_D1.4mm_L8.5mm_W2.8mm_FlatFork" H 10800 1050 50  0001 C CNN
+F 3 "https://www.mouser.com/ProductDetail/Kobiconn/151-103-RC?qs=RH7ho1lbOmmmFptH%252BQFkig%3D%3D" H 10800 1050 50  0001 C CNN
+	1    10600 1050
 	0    1    1    0
 $EndComp
@@
 F 0 "TP6" V 10604 2588 50  0000 L CNN
 F 1 "TestPoint" V 10695 2588 50  0000 L CNN
-F 2 "" H 10850 2400 50  0001 C CNN
+F 2 "Connector_Pin:Pin_D1.4mm_L8.5mm_W2.8mm_FlatFork" H 10850 2400 50  0001 C CNN
 F 3 "~" H 10850 2400 50  0001 C CNN
 	1    10650 2400
@@
 F 0 "TP2" H 5008 2618 50  0000 L CNN
 F 1 "TestPoint" H 5008 2527 50  0000 L CNN
-F 2 "" H 5150 2500 50  0001 C CNN
+F 2 "Connector_Pin:Pin_D1.4mm_L8.5mm_W2.8mm_FlatFork" H 5150 2500 50  0001 C CNN
 F 3 "~" H 5150 2500 50  0001 C CNN
 	1    4950 2500
@@
 F 0 "TP4" V 5204 3538 50  0000 L CNN
 F 1 "TestPoint" V 5295 3538 50  0000 L CNN
-F 2 "" H 5450 3350 50  0001 C CNN
+F 2 "Connector_Pin:Pin_D1.4mm_L8.5mm_W2.8mm_FlatFork" H 5450 3350 50  0001 C CNN
 F 3 "~" H 5450 3350 50  0001 C CNN
 	1    5250 3350
@@
 F 0 "TP3" V 5204 1938 50  0000 L CNN
 F 1 "TestPoint" V 5295 1938 50  0000 L CNN
-F 2 "" H 5450 1750 50  0001 C CNN
+F 2 "Connector_Pin:Pin_D1.4mm_L8.5mm_W2.8mm_FlatFork" H 5450 1750 50  0001 C CNN
 F 3 "~" H 5450 1750 50  0001 C CNN
 	1    5250 1750
@@
 F 0 "TP1" H 5008 1118 50  0000 L CNN
 F 1 "TestPoint" H 5008 1027 50  0000 L CNN
-F 2 "" H 5150 1000 50  0001 C CNN
+F 2 "Connector_Pin:Pin_D1.4mm_L8.5mm_W2.8mm_FlatFork" H 5150 1000 50  0001 C CNN
 F 3 "~" H 5150 1000 50  0001 C CNN
 	1    4950 1000
@@
 Wire Wire Line
 	650  5850 650  5800
+Text GLabel 8650 3850 0    50   Input ~ 0
+V_in
+Wire Wire Line
+	8650 3850 8650 3950
 $EndSCHEMATC
