File: charger/charger.kicad_pcb (KiCad board)
At the start: 2 copper layers, 105 parts, among them J1 OSTT7020150, J2 Conn_01x06, J3 Conn_01x06, J4 Conn_01x03, J5 OSTT7020150, Q1 CSD18540Q5B, Q2 CSD19531Q5A, Q3 CSD19531Q5A, Q4 CSD19531Q5A, Q5 CSD19531Q5A, Q6 CSD18540Q5B, U1 MSP432, U2 NCP718xSN500, U3 UCC27517DBVR, U4 INA240A2PW, U5 LM5109BMA, U6 LM5109BMA, U7 INA240A2PW, U8 LM5009MM, U9 AP131-33

Commit message: finished pcb
Parts:
- R24: footprint Resistor_SMD:R_1206_3216Metric -> Resistor_SMD:R_2512_6332Metric
- moved C18 113.3 mm to (54.6, 45.7)
- moved C21 113.3 mm to (54.6, 43.2)
- moved U4 113.3 mm to (47.4, 43.5)
- moved R11 113.3 mm to (54.6, 40.6)
- moved FB1 113.3 mm to (49.5, 47.0)
- moved C8 108.9 mm to (61.0, 35.6), turned to 270 degrees
- moved R6 107.2 mm to (58.4, 35.6), turned to 270 degrees
- moved R5 105.7 mm to (55.9, 35.6), turned to 90 degrees
- moved C22 35.6 mm to (221.0, 91.4), turned to 180 degrees
- moved R24 33.7 mm to (232.4, 41.9)
- moved R19 30.5 mm to (221.0, 94.0), turned to 180 degrees
- moved R18 25.4 mm to (221.0, 96.5), turned to 0 degrees
- moved R2 20.9 mm to (223.5, 152.4), turned to 90 degrees
- moved J4 15.3 mm to (238.8, 143.5), turned to 0 degrees
- moved J3 12.7 mm to (238.8, 134.6)
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- renumbered 10V to TP5, 3V3 to TP6, 5V to TP7
Routing:
- net GND: track 0.00 -> 346.3 mm, vias 0 -> 24
- net V_in_sense: track 0.00 -> 315.1 mm
- net I_in_sense: track 2.54 -> 313.3 mm, vias 0 -> 1
- net +3V3: track 0.00 -> 302.9 mm, vias 0 -> 6
- net +10V: track 4.17 -> 214.1 mm, vias 0 -> 8
- net +5V: track 0.00 -> 183.3 mm
- net Input_EN: track 0.00 -> 142.4 mm, vias 0 -> 3
- net V_bat_sense: track 0.00 -> 128.6 mm, vias 0 -> 1
- net I_bat_sense: track 2.54 -> 118.9 mm
- net SPI_CS_WL: track 0.00 -> 89.5 mm
- net G1_H: track 0.00 -> 87.2 mm, vias 0 -> 2
- net +Bat: track 0.00 -> 82.8 mm, vias 0 -> 3
- net SPI_MOSI: track 0.00 -> 80.9 mm
- net V_out: track 0.00 -> 78.8 mm
- net G2_H: track 0.00 -> 78.0 mm, vias 0 -> 2
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- added copper zone on B.Cu, net +Bat
- added copper zone on F.Cu, net +Bat
- added copper zone on F.Cu, net -Bat
- added copper zone on B.Cu, net GND
- added copper zone on F.Cu, net GND
- added copper zone on F.Cu, net Net-(L1-Pad1)
- added copper zone on F.Cu, net Net-(L2-Pad1)
- added copper zone on F.Cu, net V_out
- added copper zone on F.Cu, net V_solar
- added copper zone on F.Cu, net V_solar-

Commit message: charger pcb v2
Parts:
- removed the C15 at (171.4, 48.3)
- removed the C32 at (59.7, 67.3)
- removed the C33 at (47.0, 66.0)
- removed the C35 at (57.1, 80.0)
- removed the J2 at (213.4, 157.5)
- removed J4: Conn_01x03, Connector_PinHeader_2.54mm:PinHeader_1x03_P2.54mm_Vertical
- removed R2, R30: 1k, Resistor_SMD:R_1206_3216Metric
- removed R27, R28: 0 ohm, Resistor_SMD:R_1206_3216Metric
- removed R29: 3k, Resistor_SMD:R_1206_3216Metric
- removed R31: 3, Resistor_SMD:R_1206_3216Metric
- removed TP1, TP2: TestPoint, Connector_Pin:Pin_D1.4mm_L8.5mm_W2.8mm_FlatFork
- removed the U1 at (156.2, 153.7)
- removed the U8 at (53.3, 68.6)
- added C11: 560u, Capacitor_SMD:C_Elec_8x10.2, F.Cu at (223.4, 121.8)
- added C21: 0.1 uF, Capacitor_SMD:C_1206_3216Metric, B.Cu at (179.1, 145.4)
- added C22: 0.1 uF, Capacitor_SMD:C_1206_3216Metric, B.Cu at (174.0, 149.2)
- added C31: 0.1 uF, Capacitor_SMD:C_1206_3216Metric, B.Cu at (128.3, 119.4)
- added C37: 120u, Capacitor_SMD:C_Elec_10x10.2, F.Cu at (114.3, 103.5)
- added U6: LM321, Package_TO_SOT_SMD:SOT-23-5, B.Cu at (133.3, 137.8)
- added U7: LM321, Package_TO_SOT_SMD:SOT-23-5, F.Cu at (153.7, 32.4)
- added U9: LM2594HVM-12, Package_SO:SOIC-8_3.9x4.9mm_P1.27mm, B.Cu at (118.1, 117.5)
- C10: renamed from C11; moved to B.Cu
- C12: value 560 uF -> 560u; footprint Capacitor_SMD:C_1206_3216Metric -> Capacitor_SMD:C_Elec_8x10.2
- C13: value 560 uF -> 220u; footprint Capacitor_SMD:C_1206_3216Metric -> Capacitor_SMD:C_Elec_6.3x7.7
- C14: value 220 uF -> 220u; footprint Capacitor_SMD:C_1206_3216Metric -> Capacitor_SMD:C_Elec_6.3x7.7
- C17: renamed from C8; moved to B.Cu
- C28: renamed from C26; moved to B.Cu
- C29: renamed from C28; moved to B.Cu
- C30: value 1 uF -> 68u; footprint Capacitor_SMD:C_1206_3216Metric -> Capacitor_SMD:C_Elec_8x10.2
- C33: renamed from C1; moved to B.Cu
- C34, D5, FB1, Q1, Q2, Q3, Q4, Q5, Q6: moved to B.Cu
- C35: renamed from C2; moved to B.Cu
- C4: renamed from C6; moved to B.Cu
- C5: renamed from C7; moved to B.Cu
- C6: renamed from C18; moved to B.Cu
- C7: renamed from C9; moved to B.Cu
- C8: renamed from C10; moved to B.Cu
- C9: renamed from C21; moved to B.Cu
- D6: value B1100B -> MBRS140T3G; footprint Diode_SMD:D_SMB -> Diode_SMD:D_SMB_Handsoldering
- J1: footprint Connector_PinHeader_2.54mm:PinHeader_1x06_P2.54mm_Vertical -> MWD_Footprints:Phoenix_MKDS_6.35
- J2: renamed from J5; footprint Connector_PinHeader_2.54mm:PinHeader_1x02_P2.54mm_Vertical -> MWD_Footprints:Phoenix_MKDS_6.35
- J3: value Conn_01x06 -> MECF-50-01-X-DV; footprint Connector_PinHeader_2.54mm:PinHeader_1x06_P2.54mm_Vertical -> MECF-50-01-X-DV:SAMTEC_MECF-50-01-X-DV
- L3: value 220 uH -> 330 uH
- R10: renamed from R5; value 950k -> 698k; moved to B.Cu
- R11: renamed from R6; moved to B.Cu
- R12: renamed from R18; value 1M -> 806k
- R25: value 430k -> 47k; moved to B.Cu
- R26: value 169k -> 47k; moved to B.Cu
- R3: footprint Resistor_SMD:R_1206_3216Metric -> Resistor_SMD:R_2512_6332Metric; moved to B.Cu
- R5: renamed from R11; moved to B.Cu
- U10: renamed from U2; moved to B.Cu
- U11: renamed from U9; moved to B.Cu
- U3: renamed from U4; footprint Package_SO:TSSOP-8_4.4x3mm_P0.65mm -> Package_SO:SOIC-8_3.9x4.9mm_P1.27mm; moved to B.Cu
- U8: renamed from U7; footprint Package_SO:TSSOP-8_4.4x3mm_P0.65mm -> Package_SO:SOIC-8_3.9x4.9mm_P1.27mm
- moved C5 143.8 mm to (188.0, 117.6), turned to 90 degrees
- moved C7 140.3 mm to (185.4, 117.6), turned to 90 degrees
- moved C3 138.1 mm to (200.7, 113.0), turned to 180 degrees
- moved C8 136.7 mm to (182.9, 117.6), turned to 90 degrees
- moved C10 133.2 mm to (180.3, 117.6), turned to 90 degrees
- moved C4 129.7 mm to (177.8, 117.6), turned to 90 degrees
- moved R15 128.8 mm to (218.7, 103.5)
- moved C17 128.3 mm to (138.4, 137.8), turned to 0 degrees
- moved R11 127.8 mm to (138.4, 135.3), turned to 0 degrees
- moved R10 127.5 mm to (138.4, 132.7), turned to 180 degrees
- moved C15 122.7 mm to (206.4, 125.1), turned to 270 degrees
- moved C19 122.4 mm to (214.0, 106.7), turned to 0 degrees
- moved D1 121.7 mm to (210.2, 120.0)
- moved Q2 120.2 mm to (218.4, 95.2), turned to 0 degrees
- moved R8 116.5 mm to (207.4, 129.8)
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- renumbered C3 to C1, C16 to C15, C17 to C16, C22 to C18, C4 to C2, C27 to C26, C29 to C27, C5 to C3, C31 to C32, R19 to R13, R12 to R14, R13 to R15, R14 to R16, R15 to R17, R16 to R18, R17 to R19, R23 to R22, R22 to R23, R7 to R6, R8 to R7, R9 to R8, R10 to R9, U3 to U1, U5 to U4, U6 to U5
Connections:
- C1 pad 2: +10V -> +12V
- C12 pad 1: GND -> /PWM_L2
- C12 pad 2: /PWM_L1 -> GND
- C13 pad 1: GND -> /PWM_H1
- C13 pad 2: /PWM_L2 -> GND
- C14 pad 1: /PWM_H1 -> /PWM_H2
- C15 pad 2: +10V -> +12V
- C16 pad 2: +10V -> +12V
- C17 pad 1: V_in_sense -> Net-(C17-Pad1)
- C18 pad 1: V_bat_sense -> Net-(C18-Pad1)
- C30 pad 1: GND -> V_in
- C30 pad 2: V_in -> GND
- C33 pad 1: +10V -> +12V
- D1 pad 2: +10V -> +12V
- D2 pad 2: +10V -> +12V
- J1 pad 1: V_solar -> V_solar-
- J1 pad 2: /SP1- -> V_solar
- J3 pad 1: SPI_CLK -> +3V3
- J3 pad 2: SPI_CS_WL -> Net-(J3-Pad2)
- J3 pad 3: SPI_MOSI -> +3V3
- J3 pad 4: SPI_MISO -> Net-(J3-Pad4)
- J3 pad 5: SPI_CS_D -> +3V3
- J3 pad 6: GND -> Net-(J3-Pad6)
- L1 pad 1: Net-(L1-Pad1) -> V_out
- L1 pad 2: V_out -> Net-(L1-Pad2)
- L3 pad 2: Net-(L3-Pad2) -> +12V
- Q2 pad 1: Net-(L1-Pad1) -> Net-(L1-Pad2)
- Q2 pad 2: Net-(L1-Pad1) -> Net-(L1-Pad2)
- Q2 pad 3: Net-(L1-Pad1) -> Net-(L1-Pad2)
- Q3 pad 5: Net-(L1-Pad1) -> Net-(L1-Pad2)
- R10 pad 2: V_in_sense -> Net-(C17-Pad1)
- R11 pad 1: V_in_sense -> Net-(C17-Pad1)
- R12 pad 2: V_bat_sense -> Net-(C18-Pad1)
- R13 pad 1: V_bat_sense -> Net-(C18-Pad1)
- R15 pad 1: Net-(L1-Pad1) -> Net-(L1-Pad2)
- R20 pad 1: Net-(L1-Pad1) -> Net-(L1-Pad2)
- R25 pad 2: V_in -> Net-(C31-Pad2)
- R26 pad 1: Net-(R26-Pad1) -> GND
- R26 pad 2: Net-(R26-Pad2) -> Net-(R25-Pad1)
- TP5 pad 1: +10V -> +12V
- U1 pad 1: +10V -> +12V
- U10 pad 1: +10V -> +12V
- U10 pad 3: Net-(R27-Pad1) -> +12V
- U11 pad 3: Net-(R28-Pad2) -> +5V
- U4 pad 1: +10V -> +12V
- U5 pad 1: +10V -> +12V
Routing:
- net V_in_sense: track 315.1 -> 53.0 mm, vias 0 -> 1
- net +12V: track 0.00 -> 243.9 mm, vias 0 -> 5
- net +10V: track 214.1 -> 0.00 mm, vias 8 -> 0
- net GND: track 346.3 -> 143.7 mm, vias 24 -> 78
- net I_in_sense: track 313.3 -> 113.2 mm, vias 1 -> 3
- net +5V: track 183.3 -> 26.4 mm
- net SPI_CS_WL: track 89.5 -> 0.00 mm
- net V_bat_sense: track 128.6 -> 215.3 mm, vias 1 -> 4
- net SPI_MOSI: track 80.9 -> 0.00 mm
- net SPI_CLK: track 77.4 -> 0.00 mm
- net SPI_MISO: track 76.6 -> 0.00 mm
- net SPI_CS_D: track 72.3 -> 0.00 mm
- net I_bat_sense: track 118.9 -> 191.0 mm, vias 0 -> 4
- net I2C_SCL: track 67.2 -> 0.00 mm
- net I2C_SDA: track 65.0 -> 0.00 mm
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- added copper zone on B.Cu, net -Bat
- added copper zone on B.Cu, net Net-(L1-Pad2)
- added copper zone on F.Cu, net Net-(L1-Pad2)
- added copper zone on B.Cu, net Net-(L2-Pad1)
- added copper zone on B.Cu, net V_in
- added copper zone on B.Cu, net V_solar
- added copper zone on B.Cu, net V_solar-
- removed copper zone on B.Cu, net +Bat
- removed copper zone on F.Cu, net -Bat
- removed copper zone on F.Cu, net Net-(L1-Pad1)
- removed copper zone on F.Cu, net V_in
- removed copper zone on F.Cu, net V_solar
- removed copper zone on F.Cu, net V_solar-
Other:
- board outline added: 125.7 x 134.6 mm
- board text added: "Mark Ditsworth"
- board text added: "Solar Panel Battery Charger Version 2.1"
